File: kicad_design_files/bldc_driver/bldc_driver.kicad_pcb (KiCad board)
At the start: 4 copper layers, 1.3 x 7.5 mm, 66 parts, among them J1 TBP01R1-508-02BE, J2 TBP01R1-508-03BE, J3 530480210, J4 530480510, J5 USB3130-XX-X_REVD, Q1 DMN6040SK3-13, Q2 DMN6040SK3-13, Q3 DMN6040SK3-13, Q4 DMN6040SK3-13, Q5 DMN6040SK3-13, Q6 DMN6040SK3-13, Q7 SS8050-G, Q8 SS8050-G, U1 AZ1117ID-3.3TRG1, U2 SMF05CT1G, U3 ESP32-WROOM-32U, U4 AZ1117ID-3.3TRG1, U5 CP2102-GMR-QFN28, U6 TMC6200-TA-T

Commit message: Done
Parts:
- C15, Q1, Q6, R4, R5, R6: moved to B.Cu
- H1, H2, H3, H4: value MountingHole -> MountingHole_Pad; footprint MountingHole:MountingHole_3.2mm_M3 -> MountingHole:MountingHole_3.2mm_M3_DIN965_Pad
- Q2: renamed from Q4; moved to B.Cu
- Q3: renamed from Q2; moved to B.Cu
- Q4: renamed from Q5; moved to B.Cu
- Q5: renamed from Q3; moved to B.Cu
- moved J2 139.7 mm to (146.6, 100.2), turned to -90 degrees
- moved H4 99.5 mm to (145.3, 128.5)
- moved H3 94.3 mm to (87.4, 128.5)
- moved J1 86.9 mm to (85.8, 115.8), turned to 90 degrees
- moved C14 76.4 mm to (95.8, 112.8), turned to 90 degrees
- moved C2 74.9 mm to (121.9, 105.2), turned to 90 degrees
- moved R1 70.9 mm to (110.6, 111.5), turned to -90 degrees
- moved LED1 68.6 mm to (109.0, 111.5), turned to -90 degrees
- moved C15 66.6 mm to (99.3, 113.5), turned to 90 degrees
- moved J3 65.9 mm to (122.0, 64.7), turned to 180 degrees
- moved C1 64.4 mm to (115.3, 110.2), turned to 0 degrees
- moved U1 63.8 mm to (113.8, 105.2), turned to 90 degrees
- moved R4 61.9 mm to (129.8, 117.8)
- moved R2 57.8 mm to (120.1, 70.1)
- moved R3 57.6 mm to (123.2, 70.1)
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Connections:
- net /PHASEU renamed /PHASE_U
- net /PHASEW renamed /PHASE_W
- J2 pad 2: /PHASEV -> /PHASE_V
- Q7 pad 2: /esp32/ESP_IO0 -> /esp32/DTR
- Q7 pad 3: /esp32/DTR -> /esp32/ESP_IO0
- Q8 pad 1: Net-(Q8-Pad1) -> Net-(R9-Pad2)
- R8 pad 1: /esp32/DTR -> /esp32/ESP_IO0
- R8 pad 2: Net-(Q8-Pad1) -> +3.3V
- R9 pad 1: /esp32/ESP_IO0 -> /esp32/DTR
- R9 pad 2: +3.3V -> Net-(R9-Pad2)
Routing:
- net +3.3V: track 0.00 -> 175.9 mm, vias 0 -> 3
- net /CURW: track 0.00 -> 86.5 mm, vias 0 -> 2
- net /CURV: track 0.00 -> 81.4 mm, vias 0 -> 2
- net /LV: track 0.00 -> 78.4 mm, vias 0 -> 3
- net GND: track 0.00 -> 77.3 mm, vias 0 -> 38
- net /LW: track 0.00 -> 72.7 mm, vias 0 -> 1
- net +12V: track 0.00 -> 72.1 mm, vias 0 -> 2
- net /HV: track 0.00 -> 61.5 mm, vias 0 -> 1
- net /HW: track 0.00 -> 59.4 mm, vias 0 -> 3
- net /HU: track 0.00 -> 54.6 mm, vias 0 -> 3
- net /V: track 0.00 -> 53.0 mm, vias 0 -> 3
- net /FAULT: track 0.00 -> 52.9 mm, vias 0 -> 2
- net /DRV_EN: track 0.00 -> 52.3 mm, vias 0 -> 2
- net /LU: track 0.00 -> 51.2 mm, vias 0 -> 3
- net /CURU: track 0.00 -> 48.7 mm, vias 0 -> 3
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- added copper zone on B.Cu, net (none)
- added copper zone on F.Cu, net +3.3V
- added copper zone on B.Cu, net /PHASE_V
- added copper zone on B.Cu, net /PHASE_W
- added copper zone on B.Cu, net /U
- added copper zone on B.Cu, net /V
- added copper zone on B.Cu, net /VIN
- added copper zone on B.Cu, net /W
- added copper zone on B.Cu, net GND
- added copper zone on F.Cu, net GND
Other:
- board size 1.3 x 7.5 mm -> 66.3 x 70.3 mm
- copper layers 4 -> 2
