File: kicad_design_files/bldc_driver/esp32.kicad_sch (KiCad schematic)
At the start: 23 parts, among them J5 USB3130-XX-X_REVD, Q7 SS8050-G, Q8 SS8050-G, U2 SMF05CT1G, U3 ESP32-WROOM-32U, U4 AZ1117ID-3.3TRG1, U5 INTERFACE-CP2102-GMR_QFN28_

Commit message: Done
Parts:
- C6: value 10uF_6.3V_X5R_±20%_0402 -> 10uF_6.3V_0402
Connections:
- net +3.3V: now also R8.2; no longer R9.2
- net DTR: now also Q7.2, R9.1; no longer Q7.3, R8.1
- net ESP_IO0: now also Q7.3, R8.1; no longer Q7.2, R9.1
- net at Q8.1: now also R9.2; no longer R8.2
Other:
- moved on the sheet: C6, Q8, R11, R9
